File: leds.sch (KiCad schematic (older format))
At the start: 75 parts

Commit message: Add LEDs under each key
Changed lines of the file:
@@
 	750  5200 1150 5200
 Connection ~ 1150 5200
-Text GLabel 3850 1150 2    50   Input ~ 0
+Text HLabel 3850 1150 2    50   Input ~ 0
 LED
 $EndSCHEMATC

Commit message: Move PCB references
Connections:
- no-connect marks 0 -> 1
Changed lines of the file:
@@
 Text HLabel 3850 1150 2    50   Input ~ 0
 LED
+NoConn ~ 6850 4900
 $EndSCHEMATC
