File: undiscipline-noled/undiscipline-noled.kicad_pcb (KiCad board)
At the start: 4 copper layers, 337.8 x 133.5 mm, 181 parts, among them J2 USB_B_Micro, SW1 SW_Push, SW10 SW_Push, SW11 SW_Push, SW12 SW_Push, SW13 SW_Push, SW14 SW_Push, SW15 SW_Push, SW16 SW_Push, SW17 SW_Push, SW18 SW_Push, SW19 SW_Push, SW2 SW_Push, SW20 SW_Push, SW21 SW_Push, SW22 SW_Push, SW23 SW_Push, SW24 SW_Push, SW25 SW_Push, SW26 SW_Push, SW27 SW_Push, SW28 SW_Push, SW29 SW_Push, SW3 SW_Push, SW30 SW_Push, SW31 SW_Push, SW32 SW_Push, SW33 SW_Push, SW34 SW_Push, SW35 SW_Push, SW36 SW_Push, SW37 SW_Push, SW38 SW_Push, SW39 SW_Push, SW4 SW_Push, SW40 SW_Push, SW41 SW_Push, SW42 SW_Push, SW43 SW_Push, SW44 SW_Push, SW45 SW_Push, SW46 SW_Push, SW47 SW_Push, SW48 SW_Push, SW49 SW_Push, SW5 SW_Push, SW50 SW_Push, SW51 SW_Push, SW52 SW_Push, SW53 SW_Push, SW54 SW_Push, SW55 SW_Push, SW56 SW_Push, SW57 SW_Push, SW58 SW_Push, SW59 SW_Push, SW6 SW_Push, SW60 SW_Push, SW61 SW_Push, SW62 SW_Push, SW63 SW_Push, SW64 SW_Push, SW65 SW_Push, SW66 SW_Push, SW67 SW_Push, SW68 SW_Push, SW69 SW_Push, SW7 SW_Push, SW70 SW_Push, SW71 SW_Push, SW72 SW_Push, SW73 SW_Push, SW74 SW_Push, SW75 SW_Push, SW8 SW_Push, SW9 SW_Push, U1 ATmega32A-PU, Y1 16MHz

Commit message: Redesign the whole noled layout
Parts:
- removed REF** (x4): MountingHole_2.2mm_M2, MountingHole:MountingHole_2.2mm_M2
- moved H9 40.4 mm to (209.4, 208.4)
- moved R3 26.4 mm to (305.8, 92.0)
- moved H11 21.5 mm to (258.3, 83.7)
- moved H10 21.5 mm to (258.3, 106.5)
- moved H6 21.2 mm to (377.2, 106.5)
- moved H5 21.1 mm to (377.2, 83.7)
- moved C1 20.9 mm to (360.2, 106.0)
- moved C2 20.9 mm to (344.7, 106.0)
- moved D76 20.9 mm to (286.0, 91.5)
- moved D77 20.9 mm to (286.0, 95.1)
- moved J2 20.9 mm to (295.0, 79.7)
- moved R4 20.9 mm to (305.8, 83.4)
- moved U1 20.9 mm to (322.9, 99.7)
- moved Y1 20.9 mm to (354.9, 104.8)
- moved SW_BOOT1 20.9 mm to (277.5, 83.7)
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Routing:
- net +5V: track 116.6 -> 64.7 mm
- net col1: track 370.3 -> 364.5 mm
- net col5: track 244.6 -> 250.4 mm
- net row4: track 414.5 -> 419.6 mm
- net col0: track 391.6 -> 386.6 mm
- net col3: track 341.7 -> 337.4 mm
- net col10: track 197.8 -> 193.8 mm
- net col4: track 303.0 -> 299.3 mm
- net col8: track 190.5 -> 194.0 mm
- net row2: track 383.4 -> 386.5 mm
- net col2: track 333.0 -> 329.9 mm
- net col7: track 233.4 -> 236.3 mm
- net Net-(D77-Pad1): track 29.3 -> 26.4 mm
- net row0: track 283.0 -> 285.8 mm
- net col11: track 178.8 -> 176.7 mm
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Other:
- board size 337.8 x 133.5 mm -> 343.6 x 132.8 mm

Commit message: Update uv mask
Parts:
- C5: moved to F.Cu
- moved C4 2.47 mm to (341.5, 101.0), turned to 270 degrees
- moved D76 1.45 mm to (286.0, 90.1)
- moved D77 1.45 mm to (286.0, 93.6)
- moved H11 1.45 mm to (258.3, 82.2)
- moved H2 1.45 mm to (41.6, 82.2)
- moved H3 1.45 mm to (157.5, 82.2)
- moved H5 1.45 mm to (377.2, 82.2)
- moved J2 1.45 mm to (295.0, 78.2)
- moved U1 1.45 mm to (322.9, 98.3)
- moved C1 1.45 mm to (360.2, 104.6)
- moved C2 1.45 mm to (344.7, 104.6)
- moved C5 1.45 mm to (348.2, 80.2)
- moved H10 1.45 mm to (258.3, 105.1)
- moved H4 1.45 mm to (41.6, 105.1)
- moved H6 1.45 mm to (377.2, 105.1)
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Routing:
- net col5: track 250.4 -> 245.9 mm
- net reset: track 92.2 -> 89.6 mm
- net col8: track 194.0 -> 196.4 mm
- net col9: track 177.5 -> 179.9 mm
- net col13: track 143.2 -> 145.3 mm
- net col15: track 94.0 -> 95.4 mm
- net col7: track 236.3 -> 234.9 mm
- net col11: track 176.7 -> 178.1 mm
- net col10: track 193.8 -> 195.1 mm
- net col12: track 95.6 -> 96.8 mm
- net row3: track 399.7 -> 400.6 mm
- net row4: track 419.6 -> 420.6 mm
- net row5: track 447.5 -> 448.4 mm
- net row1: track 370.7 -> 371.5 mm
- net row2: track 386.5 -> 387.3 mm
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Other:
- board size 343.6 x 132.8 mm -> 343.6 x 134.2 mm

Commit message: Add plates
Parts:
- removed H10, H11, H7, H8, H9: MountingHole_Pad, MountingHole:MountingHole_2.2mm_M2_DIN965_Pad_TopBottom
- added REF**: MountingHole_2.2mm_M2, MountingHole:MountingHole_2.2mm_M2, F.Cu at (372.6, 164.8)
- added REF**: MountingHole_2.2mm_M2, MountingHole:MountingHole_2.2mm_M2, F.Cu at (146.9, 61.4)
- added REF**: MountingHole_2.2mm_M2, MountingHole:MountingHole_2.2mm_M2, F.Cu at (146.9, 38.6)
- added REF**: MountingHole_2.2mm_M2, MountingHole:MountingHole_2.2mm_M2, F.Cu at (37.0, 38.6)
- added REF**: MountingHole_2.2mm_M2, MountingHole:MountingHole_2.2mm_M2, F.Cu at (204.8, 164.8)
- added REF**: MountingHole_2.2mm_M2, MountingHole:MountingHole_2.2mm_M2, F.Cu at (37.0, 164.8)
- added REF**: MountingHole_2.1mm, MountingHole:MountingHole_2.1mm, F.Cu at (372.6, 67.4)
- SW1, SW10, SW11, SW12, SW13, SW14, SW15, SW16, SW17, SW18, SW2, SW20, SW21, SW23, SW24, SW25, SW26, SW27, SW28, SW29, SW3, SW30, SW31, SW32, SW33, SW34, SW36, SW37, SW39, SW4, SW40, SW41, SW42, SW43, SW44, SW45, SW46, SW47, SW48, SW49, SW5, SW51, SW52, SW53, SW54, SW55, SW56, SW57, SW58, SW59, SW6, SW60, SW61, SW62, SW63, SW65, SW7, SW73, SW74, SW75, SW8, SW9: footprint keyboard-parts:CherryMX_Kailh_Socket -> Button_Switch_Keyboard:SW_Cherry_MX_1.00u_Plate
- SW19: footprint keyboard-parts:CherryMX_Kailh_Socket -> Button_Switch_Keyboard:SW_Cherry_MX_2.00u_Plate
- SW22, SW35: footprint keyboard-parts:CherryMX_Kailh_Socket -> Button_Switch_Keyboard:SW_Cherry_MX_1.50u_Plate
- SW38: footprint keyboard-parts:CherryMX_Kailh_Socket -> Button_Switch_Keyboard:SW_Cherry_MX_1.75u_Plate
- SW50: footprint keyboard-parts:CherryMX_Kailh_Socket -> Button_Switch_Keyboard:SW_Cherry_MX_2.25u_Plate
- SW64: footprint keyboard-parts:CherryMX_Kailh_Socket -> Button_Switch_Keyboard:SW_Cherry_MX_2.75u_Plate
- SW66, SW67, SW68, SW69, SW71, SW72: footprint keyboard-parts:CherryMX_Kailh_Socket -> Button_Switch_Keyboard:SW_Cherry_MX_1.25u_Plate
- SW70: footprint keyboard-parts:CherryMX_Kailh_Socket -> Button_Switch_Keyboard:SW_Cherry_MX_6.25u_Plate
- moved H4 216.5 mm to (253.7, 61.4)
- moved H1 203.6 mm to (153.8, 38.6)
- moved H2 114.1 mm to (153.8, 61.4)
- moved H3 105.7 mm to (253.7, 38.6)
- moved SW22 48.8 mm to (57.3, 87.8)
- moved SW23 48.8 mm to (81.1, 87.8)
- moved SW24 48.8 mm to (100.2, 87.8)
- moved SW25 48.8 mm to (119.2, 87.8)
- moved SW26 48.8 mm to (138.3, 87.8)
- moved SW27 48.8 mm to (157.3, 87.8)
- moved SW28 48.8 mm to (176.4, 87.8)
- moved SW29 48.8 mm to (195.4, 87.8)
- moved SW30 48.8 mm to (214.5, 87.8)
- moved SW31 48.8 mm to (233.5, 87.8)
- moved SW32 48.8 mm to (252.6, 87.8)
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Connections:
- SW1 pad 1: Net-(D1-Pad2) -> col0
- SW1 pad 2: col0 -> Net-(D1-Pad2)
- SW10 pad 1: Net-(D10-Pad2) -> col4
- SW10 pad 2: col4 -> Net-(D10-Pad2)
- SW11 pad 1: Net-(D11-Pad2) -> col5
- SW11 pad 2: col5 -> Net-(D11-Pad2)
- SW12 pad 1: Net-(D12-Pad2) -> col6
- SW12 pad 2: col6 -> Net-(D12-Pad2)
- SW13 pad 1: Net-(D13-Pad2) -> col7
- SW13 pad 2: col7 -> Net-(D13-Pad2)
- SW14 pad 1: Net-(D14-Pad2) -> col8
- SW14 pad 2: col8 -> Net-(D14-Pad2)
- SW15 pad 1: Net-(D15-Pad2) -> col9
- SW15 pad 2: col9 -> Net-(D15-Pad2)
- SW16 pad 1: Net-(D16-Pad2) -> col10
- SW16 pad 2: col10 -> Net-(D16-Pad2)
- SW17 pad 1: Net-(D17-Pad2) -> col11
- SW17 pad 2: col11 -> Net-(D17-Pad2)
- SW18 pad 1: Net-(D18-Pad2) -> col12
- SW18 pad 2: col12 -> Net-(D18-Pad2)
- SW19 pad 1: Net-(D19-Pad2) -> col13
- SW19 pad 2: col13 -> Net-(D19-Pad2)
- SW2 pad 1: Net-(D2-Pad2) -> col1
- SW2 pad 2: col1 -> Net-(D2-Pad2)
- SW20 pad 1: Net-(D20-Pad2) -> col14
- SW20 pad 2: col14 -> Net-(D20-Pad2)
- SW21 pad 1: Net-(D21-Pad2) -> col15
- SW21 pad 2: col15 -> Net-(D21-Pad2)
- SW22 pad 1: Net-(D22-Pad2) -> col0
- SW22 pad 2: col0 -> Net-(D22-Pad2)
- SW23 pad 1: Net-(D23-Pad2) -> col1
- SW23 pad 2: col1 -> Net-(D23-Pad2)
- SW24 pad 1: Net-(D24-Pad2) -> col2
- SW24 pad 2: col2 -> Net-(D24-Pad2)
- SW25 pad 1: Net-(D25-Pad2) -> col3
- SW25 pad 2: col3 -> Net-(D25-Pad2)
- SW26 pad 1: Net-(D26-Pad2) -> col4
- SW26 pad 2: col4 -> Net-(D26-Pad2)
- SW27 pad 1: Net-(D27-Pad2) -> col5
- SW27 pad 2: col5 -> Net-(D27-Pad2)
- SW28 pad 1: Net-(D28-Pad2) -> col6
- SW28 pad 2: col6 -> Net-(D28-Pad2)
- SW29 pad 1: Net-(D29-Pad2) -> col7
- SW29 pad 2: col7 -> Net-(D29-Pad2)
- SW3 pad 1: Net-(D3-Pad2) -> col2
- SW3 pad 2: col2 -> Net-(D3-Pad2)
- SW30 pad 1: Net-(D30-Pad2) -> col8
- SW30 pad 2: col8 -> Net-(D30-Pad2)
- SW31 pad 1: Net-(D31-Pad2) -> col9
- SW31 pad 2: col9 -> Net-(D31-Pad2)
- SW32 pad 1: Net-(D32-Pad2) -> col10
- SW32 pad 2: col10 -> Net-(D32-Pad2)
- SW33 pad 1: Net-(D33-Pad2) -> col11
- SW33 pad 2: col11 -> Net-(D33-Pad2)
- SW34 pad 1: Net-(D34-Pad2) -> col12
- SW34 pad 2: col12 -> Net-(D34-Pad2)
- SW35 pad 1: Net-(D35-Pad2) -> col13
- SW35 pad 2: col13 -> Net-(D35-Pad2)
- SW36 pad 1: Net-(D36-Pad2) -> col14
- SW36 pad 2: col14 -> Net-(D36-Pad2)
- SW37 pad 1: Net-(D37-Pad2) -> col15
- SW37 pad 2: col15 -> Net-(D37-Pad2)
- SW38 pad 1: Net-(D38-Pad2) -> col0
- SW38 pad 2: col0 -> Net-(D38-Pad2)
- SW39 pad 1: Net-(D39-Pad2) -> col1
- SW39 pad 2: col1 -> Net-(D39-Pad2)
- SW4 pad 1: Net-(D4-Pad2) -> col3
- SW4 pad 2: col3 -> Net-(D4-Pad2)
- SW40 pad 1: Net-(D40-Pad2) -> col2
- SW40 pad 2: col2 -> Net-(D40-Pad2)
- SW41 pad 1: Net-(D41-Pad2) -> col3
- SW41 pad 2: col3 -> Net-(D41-Pad2)
- SW42 pad 1: Net-(D42-Pad2) -> col4
- SW42 pad 2: col4 -> Net-(D42-Pad2)
- SW43 pad 1: Net-(D43-Pad2) -> col5
- SW43 pad 2: col5 -> Net-(D43-Pad2)
- SW44 pad 1: Net-(D44-Pad2) -> col6
- SW44 pad 2: col6 -> Net-(D44-Pad2)
- SW45 pad 1: Net-(D45-Pad2) -> col7
- SW45 pad 2: col7 -> Net-(D45-Pad2)
- SW46 pad 1: Net-(D46-Pad2) -> col8
- SW46 pad 2: col8 -> Net-(D46-Pad2)
- SW47 pad 1: Net-(D47-Pad2) -> col9
- SW47 pad 2: col9 -> Net-(D47-Pad2)
- SW48 pad 1: Net-(D48-Pad2) -> col10
- SW48 pad 2: col10 -> Net-(D48-Pad2)
- SW49 pad 1: Net-(D49-Pad2) -> col11
- SW49 pad 2: col11 -> Net-(D49-Pad2)
- SW5 pad 1: Net-(D5-Pad2) -> col4
- SW5 pad 2: col4 -> Net-(D5-Pad2)
- SW50 pad 1: Net-(D50-Pad2) -> col13
- SW50 pad 2: col13 -> Net-(D50-Pad2)
- SW51 pad 1: Net-(D51-Pad2) -> col14
- SW51 pad 2: col14 -> Net-(D51-Pad2)
- SW52 pad 1: Net-(D52-Pad2) -> col15
- SW52 pad 2: col15 -> Net-(D52-Pad2)
- SW53 pad 1: Net-(D53-Pad2) -> col0
- SW53 pad 2: col0 -> Net-(D53-Pad2)
- SW54 pad 1: Net-(D54-Pad2) -> col2
- SW54 pad 2: col2 -> Net-(D54-Pad2)
- SW55 pad 1: Net-(D55-Pad2) -> col3
- SW55 pad 2: col3 -> Net-(D55-Pad2)
- SW56 pad 1: Net-(D56-Pad2) -> col4
- SW56 pad 2: col4 -> Net-(D56-Pad2)
- SW57 pad 1: Net-(D57-Pad2) -> col5
- SW57 pad 2: col5 -> Net-(D57-Pad2)
- SW58 pad 1: Net-(D58-Pad2) -> col6
- SW58 pad 2: col6 -> Net-(D58-Pad2)
- SW59 pad 1: Net-(D59-Pad2) -> col7
- SW59 pad 2: col7 -> Net-(D59-Pad2)
- SW6 pad 1: Net-(D6-Pad2) -> col0
- SW6 pad 2: col0 -> Net-(D6-Pad2)
- SW60 pad 1: Net-(D60-Pad2) -> col8
- SW60 pad 2: col8 -> Net-(D60-Pad2)
- SW61 pad 1: Net-(D61-Pad2) -> col9
- SW61 pad 2: col9 -> Net-(D61-Pad2)
- SW62 pad 1: Net-(D62-Pad2) -> col10
- SW62 pad 2: col10 -> Net-(D62-Pad2)
- SW63 pad 1: Net-(D63-Pad2) -> col11
- SW63 pad 2: col11 -> Net-(D63-Pad2)
- SW64 pad 1: Net-(D64-Pad2) -> col13
- SW64 pad 2: col13 -> Net-(D64-Pad2)
- SW65 pad 1: Net-(D65-Pad2) -> col14
- SW65 pad 2: col14 -> Net-(D65-Pad2)
- SW66 pad 1: Net-(D66-Pad2) -> col0
- SW66 pad 2: col0 -> Net-(D66-Pad2)
- SW67 pad 1: Net-(D67-Pad2) -> col1
- SW67 pad 2: col1 -> Net-(D67-Pad2)
- SW68 pad 1: Net-(D68-Pad2) -> col3
- SW68 pad 2: col3 -> Net-(D68-Pad2)
- SW69 pad 1: Net-(D69-Pad2) -> col4
- SW69 pad 2: col4 -> Net-(D69-Pad2)
- SW7 pad 1: Net-(D7-Pad2) -> col1
- SW7 pad 2: col1 -> Net-(D7-Pad2)
- SW70 pad 1: Net-(D70-Pad2) -> col7
- SW70 pad 2: col7 -> Net-(D70-Pad2)
- SW71 pad 1: Net-(D71-Pad2) -> col10
- SW71 pad 2: col10 -> Net-(D71-Pad2)
- SW72 pad 1: Net-(D72-Pad2) -> col11
- SW72 pad 2: col11 -> Net-(D72-Pad2)
- SW73 pad 1: Net-(D73-Pad2) -> col13
- SW73 pad 2: col13 -> Net-(D73-Pad2)
- SW74 pad 1: Net-(D74-Pad2) -> col14
- SW74 pad 2: col14 -> Net-(D74-Pad2)
- SW75 pad 1: Net-(D75-Pad2) -> col15
- SW75 pad 2: col15 -> Net-(D75-Pad2)
- SW8 pad 1: Net-(D8-Pad2) -> col2
- SW8 pad 2: col2 -> Net-(D8-Pad2)
- SW9 pad 1: Net-(D9-Pad2) -> col3
- SW9 pad 2: col3 -> Net-(D9-Pad2)
Routing:
- net col14: track 104.8 -> 110.7 mm
- net col4: track 299.5 -> 305.0 mm
- net col2: track 330.5 -> 335.9 mm
- net col1: track 365.1 -> 370.5 mm
- net col3: track 338.0 -> 342.8 mm
- net col13: track 145.3 -> 149.9 mm
- net col7: track 234.9 -> 239.4 mm
- net col5: track 245.9 -> 250.4 mm
- net col9: track 179.9 -> 184.3 mm
- net col6: track 229.4 -> 233.9 mm
- net col11: track 178.1 -> 182.6 mm
- net col15: track 95.4 -> 99.6 mm
- net col0: track 387.2 -> 391.2 mm
- net col8: track 196.4 -> 200.1 mm
- net col12: track 96.8 -> 99.8 mm
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